File: Audio Tracking Car/Combined Signal Processor/Combined Signal Processor/Mic to Pi Entire design.brd (EAGLE design)
At the start: 160 x 100 mm, 35 parts, among them IC1 74HC153N, U1 LM339AN, U2 TL084CN

Commit message: Added pins to Vcc v.1.0.2
Parts:
- removed IC1: 74HC153N, 74xx-eu:DIL16
- removed MIC: (no value), jumper:JP2W
- added SV1: (no value), con-lstb:MA17-2
- added SV2: (no value), con-lstb:MA03-1
- added U3: SN74LS153N, SN74LS153N:DIP794W45P254L1969H508Q16
- moved CY4 1.27 mm to (-33.0, 101.6)
- moved CY5 1.27 mm to (-47.0, 101.6)
Connections:
- removed net VCC: IC1.16
- net +3V3: now also U3.16
- net +5V: now also SV2.3; no longer MIC.3
- net GND: now also SV2.2, U3.6, U3.8; no longer IC1.6, IC1.8, MIC.2
- net N$1: now also U3.7; no longer IC1.7
- net N$10: now also U3.4; no longer IC1.4
- net N$14: now also U3.3; no longer IC1.3
- net N$26: now also U3.2; no longer IC1.2
- net N$27: now also U3.14; no longer IC1.14
- net N$4: now also SV2.1; no longer MIC.1
- net N$8: now also U3.5; no longer IC1.5
