File: Audio Tracking Car/Combined Signal Processor/Combined Signal Processor/Mic to Pi Entire design.sch (EAGLE design)
At the start: 35 parts, among them IC1 74HC153N, U1 LM339AN, U2 TL084CN

Commit message: Added pins to Vcc v.1.0.2
Parts:
- removed IC1: 74HC153N, 74xx-eu:74HC153N
- removed MIC: (no value), jumper:JP2W
- removed U$1: RASPBERRY-PI_REV1, RaspberryPi:RASPBERRY-PI_REV1
- added ADC: LM339AN, LM339AN:LM339AN
- added BUCKPINS, MOTOR1, MOTOR2, VCC: (no value), pinhead:PINHD-1X2
- added D2, D3, D4, D5: LED, ngspice-simulation:LED
- added JP3: (no value), pinhead:PINHD-1X3
- added JP4: (no value), pinhead:PINHD-2X20
- added R23, R24: 69, rcl:R-US_0204/7
- added SW1: (no value), special:SW_DIP-8
- added U3: SN74LS153N, SN74LS153N:SN74LS153N
- added ULTRASONIC: (no value), pinhead:PINHD-1X55X2MM
- U1: value LM339AN -> SN754410NE; device LM339AN:LM339AN -> SN754410NE:SN754410NE
Connections:
- removed net VCC/2: U2.VCC+, U2.VCC-
- new net N$22: JP4.5, R23.1, R24.2
- new net N$23: JP4.3, ULTRASONIC.2
- new net N$28: R23.2, ULTRASONIC.3
- new net N$29: ULTRASONIC.4
- new net N$30: D2.A, JP4.15, SW1.16
- new net N$31: D3.A, JP4.19, SW1.15
- new net N$32: D4.A, JP4.21, SW1.14
- new net N$33: D5.A, JP4.23, SW1.13
- new net N$34: JP4.16, U1.1,2EN
- new net N$35: JP4.18, U1.3,4EN
- new net N$36: MOTOR1.1, U1.1Y
- new net N$37: MOTOR1.2, U1.2Y
- new net N$38: MOTOR2.1, U1.3Y
- new net N$39: MOTOR2.2, U1.4Y
- new net N$40: JP4.29, U1.1A
- new net N$41: JP4.31, U1.4A
- new net N$42: JP4.7, U1.3A
- new net N$43: U2.VCC-, VCC.2
- new net N$44: U2.VCC+, VCC.1
- net +3V3: now also JP4.1, JP4.17, SW1.1, SW1.2, SW1.3, SW1.4, U3.VCC; no longer U$1.3V3@1
- net +5V: now also ADC.VCC, BUCKPINS.1, JP3.1, JP4.2, JP4.4, U1.VCC1, U1.VCC2, ULTRASONIC.1; no longer MIC.3, U$1.5V@4, U1.VCC
- net GND: now also ADC.GND, BUCKPINS.2, D2.C, D3.C, D4.C, D5.C, JP3.2, JP4.14, JP4.20, JP4.25, JP4.30, JP4.34, JP4.39, JP4.6, JP4.9, R24.1, U3.1C0, U3.GND, ULTRASONIC.5; no longer IC1A.1C0, MIC.2, U$1.GND@14, U$1.GND@20, U$1.GND@25, U$1.GND@9, U1.GND
- net N$1: now also U3.1Y; no longer IC1A.1Y
- net N$10: now also U3.1C2; no longer IC1A.1C2
- net N$14: now also U3.1C3; no longer IC1A.1C3
- net N$15: now also ADC.IN1+, ADC.IN2+, ADC.IN3+; no longer U1.IN1+, U1.IN2+, U1.IN3+
- net N$16: now also ADC.OUT2, JP4.38; no longer U$1.GPIO8,SPI0_CE0, U1.OUT2
- net N$17: now also ADC.IN1-; no longer U1.IN1-
- net N$18: now also ADC.IN2-; no longer U1.IN2-
- net N$19: now also ADC.IN3-; no longer U1.IN3-
- net N$20: now also ADC.OUT1, JP4.36; no longer U$1.GPIO25, U1.OUT1
- net N$21: now also ADC.OUT3, JP4.40; no longer U$1.GPIO7,SPI0_CE1, U1.OUT3
- net N$26: now also JP4.35, U3.B; no longer IC1A.B, U$1.GPIO9_MISO
- net N$27: now also JP4.37, U3.A; no longer IC1A.A, U$1.GPIO11_SCLK
- net N$4: now also JP3.3; no longer MIC.1
- net N$8: now also U3.1C1; no longer IC1A.1C1
Other:
- note added: "1. Buck + 2. Buck -"
- note added: "1.Vcc 2.Trig 3.Echo 4.Out 5.GND"
- moved on the sheet: CY2, CY3, CY6, CY7, D1, R10, R11, R12, R19, R20, R7, R8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
