File: Audio Tracking Car/Combined Signal Processor/Combined Signal Processor/Mic to pi entire design without pinouts.sch (EAGLE design)
At the start: 55 parts, among them U2 TL084CN, U3 TL084CN

Commit message: Included multiple versions
Parts:
- added 3V3POWER, 5VPOWER: (no value), pinhead:PINHD-1X2
Connections:
- removed net N$29: JP4.16
- removed net N$30: JP4.18
- removed net N$40: JP4.29
- removed net N$42: JP4.7
- new net N$22: JP4.35, JP4.37
- net +3V3: now also 3V3POWER.1
- net +5V: now also 5VPOWER.1
- net GND: now also 3V3POWER.2, 5VPOWER.2
- net N$23: now also JP4.33; no longer JP4.31
