File: Audio Tracking Car/Combined Signal Processor/Combined Signal Processor/Mic to Pi Entire design including pinouts.sch (EAGLE design)
At the start: 63 parts, among them U2 TL084CN, U3 TL084CN

Commit message: Add files via upload
Parts:
- removed JP2: (no value), pinhead:PINHD-1X3
Changed lines of the file:
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@@
 <part name="SUPPLY6" library="supply2" library_urn="urn:adsk.eagle:library:372" deviceset="GND" device=""/>
 <part name="U.S." library="pinhead" library_urn="urn:adsk.eagle:library:325" deviceset="PINHD-1X5" device="5X2MM" package3d_urn="urn:adsk.eagle:package:22466/2"/>
-<part name="JP2" library="pinhead" library_urn="urn:adsk.eagle:library:325" deviceset="PINHD-1X3" device="" package3d_urn="urn:adsk.eagle:package:22458/2"/>
 <part name="5VPOWER" library="pinhead" library_urn="urn:adsk.eagle:library:325" deviceset="PINHD-1X2" device="" package3d_urn="urn:adsk.eagle:package:22435/2"/>
 <part name="P+3" library="supply1" library_urn="urn:adsk.eagle:library:371" deviceset="+5V" device=""/>
@@
 <attribute name="VALUE" x="80.01" y="330.2" size="1.778" layer="96"/>
 </instance>
-<instance part="JP2" gate="A" x="93.98" y="322.58" smashed="yes">
-<attribute name="NAME" x="87.63" y="328.295" size="1.778" layer="95"/>
-<attribute name="VALUE" x="87.63" y="314.96" size="1.778" layer="96"/>
-</instance>
 <instance part="5VPOWER" gate="G$1" x="58.42" y="337.82" smashed="yes">
