File: Audio Tracking Car/Combined Signal Processor/Combined Signal Processor/Mic to Pi Entire design including pinouts.brd (EAGLE design)
At the start: 124.4 x 100 mm, 62 parts, among them U2 TL084CN, U3 TL084CN

Commit message: new brd
Routing:
- net N$43: track 144.5 -> 146.6 mm
Changed lines of the file:
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@@
 <wire x1="83.9724" y1="68.58" x2="83.98" y2="68.58" width="0.1524" layer="1"/>
 <wire x1="153.3144" y1="96.6216" x2="153.6192" y2="96.6216" width="0.1524" layer="16"/>
-<wire x1="75.1332" y1="91.8972" x2="81.5848" y2="98.3488" width="0.1524" layer="16"/>
-<wire x1="75.1332" y1="86.4108" x2="75.1332" y2="91.8972" width="0.1524" layer="16"/>
-<wire x1="77.2668" y1="84.2772" x2="75.1332" y2="86.4108" width="0.1524" layer="16"/>
-<wire x1="77.2668" y1="79.0956" x2="77.2668" y2="84.2772" width="0.1524" layer="16"/>
-<wire x1="75.1332" y1="76.962" x2="77.2668" y2="79.0956" width="0.1524" layer="16"/>
+<wire x1="74.2442" y1="91.5162" x2="81.0768" y2="98.3488" width="0.1524" layer="16"/>
+<wire x1="74.2442" y1="89.8398" x2="74.2442" y2="91.5162" width="0.1524" layer="16"/>
+<wire x1="78.5368" y1="85.5472" x2="74.2442" y2="89.8398" width="0.1524" layer="16"/>
+<wire x1="78.5368" y1="80.3656" x2="78.5368" y2="85.5472" width="0.1524" layer="16"/>
+<wire x1="75.1332" y1="76.962" x2="78.5368" y2="80.3656" width="0.1524" layer="16"/>
 <wire x1="75.1332" y1="75.438" x2="75.1332" y2="76.962" width="0.1524" layer="16"/>
 <wire x1="75.8952" y1="74.676" x2="75.1332" y2="75.438" width="0.1524" layer="16"/>
@@
 <wire x1="84.2772" y1="97.3836" x2="86.4616" y2="97.3836" width="0.1524" layer="16"/>
 <wire x1="83.312" y1="98.3488" x2="84.2772" y2="97.3836" width="0.1524" layer="16"/>
-<wire x1="81.5848" y1="98.3488" x2="83.312" y2="98.3488" width="0.1524" layer="16"/>
+<wire x1="81.0768" y1="98.3488" x2="83.312" y2="98.3488" width="0.1524" layer="16"/>
 <wire x1="153.3144" y1="96.6216" x2="153.67" y2="96.52" width="0.1524" layer="16"/>
 </signal>
